File: client_input/client_input.sch (KiCad schematic (older format))
At the start: 28 parts, among them P1 Analog In, P10 Ribbon, P2 Analog In, P3 SS, P4 FTDI, P5 LiPo, P6 Ribbon, P7 Ribbon, P8 Ribbon, P9 Ribbon, SW1 RESET, SW2 PAIR_MODE, SW3 Bootload, SW4 DIPS_08, SW5 SPDT, U1 MCP3208, U2 MCP3208, U3 ESP-12E, U4 MCP1700-3302, U5 MCP23017, U6 MCP23017

Commit message: Final revisions, exports, panelization, and gerbers for Rev 2. Sent to Elecrow (11 August 2016).
Parts:
- added C2, C3, C4, C6, C7: 0.1uF, Capacitors_ThroughHole:C_Disc_D3_P2.5, symbol C_Small
- added C5: 10uF, Capacitors_ThroughHole:C_Radial_D5_L6_P2.5, symbol CP
Connections:
- wire segments 182 -> 197
Changed lines of the file:
@@
 L GND #PWR04
 U 1 1 577DA7AD
-P 5250 7400
-F 0 "#PWR04" H 5250 7150 50  0001 C CNN
-F 1 "GND" H 5250 7250 50  0000 C CNN
-F 2 "" H 5250 7400 50  0000 C CNN
-F 3 "" H 5250 7400 50  0000 C CNN
-	1    5250 7400
+P 5250 7600
+F 0 "#PWR04" H 5250 7350 50  0001 C CNN
+F 1 "GND" H 5250 7450 50  0000 C CNN
+F 2 "" H 5250 7600 50  0000 C CNN
+F 3 "" H 5250 7600 50  0000 C CNN
+	1    5250 7600
 	1    0    0    -1
 $EndComp
@@
 L +3V3 #PWR013
 U 1 1 57802025
-P 1950 3600
-F 0 "#PWR013" H 1950 3450 50  0001 C CNN
-F 1 "+3V3" H 1950 3740 50  0000 C CNN
-F 2 "" H 1950 3600 50  0000 C CNN
-F 3 "" H 1950 3600 50  0000 C CNN
-	1    1950 3600
+P 1950 5650
+F 0 "#PWR013" H 1950 5500 50  0001 C CNN
+F 1 "+3V3" H 1950 5790 50  0000 C CNN
+F 2 "" H 1950 5650 50  0000 C CNN
+F 3 "" H 1950 5650 50  0000 C CNN
+	1    1950 5650
 	1    0    0    -1
 $EndComp
@@
 	-1   0    0    -1
 $EndComp
-$Comp
-L +3V3 #PWR026
-U 1 1 57A323CC
-P 1950 5800
-F 0 "#PWR026" H 1950 5650 50  0001 C CNN
-F 1 "+3V3" H 1950 5940 50  0000 C CNN
-F 2 "" H 1950 5800 50  0000 C CNN
-F 3 "" H 1950 5800 50  0000 C CNN
-	1    1950 5800
-	1    0    0    -1
-$EndComp
 Text GLabel 2900 4200 2    60   Input ~ 0
 SPI_CLK
@@
 Text GLabel 2900 4500 2    60   Input ~ 0
 MOSI
-Connection ~ 1950 3600
-Wire Wire Line
-	1850 3750 1850 3600
-Wire Wire Line
-	1850 3600 2050 3600
-Wire Wire Line
-	2050 3600 2050 3750
+Connection ~ 1950 5800
+Wire Wire Line
+	1850 5950 1850 5800
+Wire Wire Line
+	1850 5800 2050 5800
+Wire Wire Line
+	2050 5800 2050 5950
 Connection ~ 1950 5050
 Connection ~ 7850 3200
@@
 	7850 3000 7850 3450
 Wire Wire Line
-	7850 3300 7950 3300
+	7400 3300 7950 3300
 Wire Wire Line
 	7850 3100 7950 3100
@@
 	5050 1150 5200 1150
 Wire Wire Line
-	6100 1150 6250 1150
+	6100 1150 6450 1150
 Wire Wire Line
 	6250 1150 6250 1050
@@
 	6100 1550 6100 1600
 Wire Wire Line
-	6100 1600 5650 1600
+	5650 1600 6450 1600
 Connection ~ 6100 1150
 Wire Wire Line
@@
 Wire Wire Line
 	6050 2400 6350 2400
-Connection ~ 1950 5800
-Wire Wire Line
-	1850 5950 1850 5800
-Wire Wire Line
-	1850 5800 2050 5800
-Wire Wire Line
-	2050 5800 2050 5950
 Connection ~ 1950 7250
 Wire Wire Line
@@
 	4900 5400 5200 5400
 Wire Wire Line
-	7850 5750 7950 5750
+	7500 5750 7950 5750
 $Comp
 L Switch_SPDT_x2 SW5
@@
 	6250 2100 6350 2100
 $Comp
-L +Vin #PWR027
+L +Vin #PWR026
 U 1 1 57A39C90
 P 8150 1000
-F 0 "#PWR027" H 8150 850 50  0001 C CNN
+F 0 "#PWR026" H 8150 850 50  0001 C CNN
 F 1 "+Vin" H 8150 1140 50  0000 C CNN
 F 2 "" H 8150 1000 50  0000 C CNN
@@
 	8950 1050 9100 1050
 $Comp
-L +Vin #PWR028
+L +Vin #PWR027
 U 1 1 57A3A63C
 P 5050 1050
-F 0 "#PWR028" H 5050 900 50  0001 C CNN
+F 0 "#PWR027" H 5050 900 50  0001 C CNN
 F 1 "+Vin" H 5050 1190 50  0000 C CNN
 F 2 "" H 5050 1050 50  0000 C CNN
@@
 	3950 1100 3950 1200
 $Comp
-L +Vin #PWR029
+L +Vin #PWR028
 U 1 1 57A3AFAC
 P 5250 6550
-F 0 "#PWR029" H 5250 6400 50  0001 C CNN
+F 0 "#PWR028" H 5250 6400 50  0001 C CNN
 F 1 "+Vin" H 5250 6690 50  0000 C CNN
 F 2 "" H 5250 6550 50  0000 C CNN
@@
 $EndComp
 $Comp
-L +BATT #PWR030
+L +BATT #PWR029
 U 1 1 57A3B668
 P 9100 950
-F 0 "#PWR030" H 9100 800 50  0001 C CNN
+F 0 "#PWR029" H 9100 800 50  0001 C CNN
 F 1 "+BATT" H 9100 1090 50  0000 C CNN
 F 2 "" H 9100 950 50  0000 C CNN
@@
 	9100 1050 9100 950
 $Comp
-L +BATT #PWR031
+L +BATT #PWR030
 U 1 1 57A3B867
 P 7350 1050
-F 0 "#PWR031" H 7350 900 50  0001 C CNN
+F 0 "#PWR030" H 7350 900 50  0001 C CNN
 F 1 "+BATT" H 7350 1190 50  0000 C CNN
 F 2 "" H 7350 1050 50  0000 C CNN
@@
 	7350 1150 7350 1050
 $Comp
-L +BATT #PWR032
+L +BATT #PWR031
 U 1 1 57A3BA7C
 P 3950 1100
-F 0 "#PWR032" H 3950 950 50  0001 C CNN
+F 0 "#PWR031" H 3950 950 50  0001 C CNN
 F 1 "+BATT" H 3950 1240 50  0000 C CNN
 F 2 "" H 3950 1100 50  0000 C CNN
@@
 Wire Wire Line
 	6100 4100 5100 4100
+$Comp
+L C_Small C7
+U 1 1 57ABEF01
+P 7500 5600
+F 0 "C7" H 7510 5670 50  0000 L CNN
+F 1 "0.1uF" H 7510 5520 50  0000 L CNN
+F 2 "Capacitors_ThroughHole:C_Disc_D3_P2.5" H 7500 5600 50  0001 C CNN
+F 3 "" H 7500 5600 50  0000 C CNN
+	1    7500 5600
+	1    0    0    -1
+$EndComp
+$Comp
+L +3V3 #PWR032
+U 1 1 57ABF167
+P 7500 5450
+F 0 "#PWR032" H 7500 5300 50  0001 C CNN
+F 1 "+3V3" H 7500 5590 50  0000 C CNN
+F 2 "" H 7500 5450 50  0000 C CNN
+F 3 "" H 7500 5450 50  0000 C CNN
+	1    7500 5450
+	1    0    0    -1
+$EndComp
+Wire Wire Line
+	7500 5450 7500 5500
+Wire Wire Line
+	7500 5750 7500 5700
+$Comp
+L C_Small C6
+U 1 1 57ABF929
+P 7400 3150
+F 0 "C6" H 7410 3220 50  0000 L CNN
+F 1 "0.1uF" H 7410 3070 50  0000 L CNN
+F 2 "Capacitors_ThroughHole:C_Disc_D3_P2.5" H 7400 3150 50  0001 C CNN
+F 3 "" H 7400 3150 50  0000 C CNN
+	1    7400 3150
+	1    0    0    -1
+$EndComp
+$Comp
+L +3V3 #PWR033
+U 1 1 57ABF92F
+P 7400 3000
+F 0 "#PWR033" H 7400 2850 50  0001 C CNN
+F 1 "+3V3" H 7400 3140 50  0000 C CNN
+F 2 "" H 7400 3000 50  0000 C CNN
+F 3 "" H 7400 3000 50  0000 C CNN
+	1    7400 3000
+	1    0    0    -1
+$EndComp
+Wire Wire Line
+	7400 3000 7400 3050
+Wire Wire Line
+	7400 3300 7400 3250
+$Comp
+L C_Small C3
+U 1 1 57ABFDCB
+P 2200 5750
+F 0 "C3" H 2210 5820 50  0000 L CNN
+F 1 "0.1uF" H 2210 5670 50  0000 L CNN
+F 2 "Capacitors_ThroughHole:C_Disc_D3_P2.5" H 2200 5750 50  0001 C CNN
+F 3 "" H 2200 5750 50  0000 C CNN
+	1    2200 5750
+	1    0    0    -1
+$EndComp
+Wire Wire Line
+	1950 5800 1950 5650
+Wire Wire Line
+	1950 5650 2200 5650
+Connection ~ 1950 5650
+$Comp
+L GND #PWR034
+U 1 1 57AC014A
+P 2200 5900
+F 0 "#PWR034" H 2200 5650 50  0001 C CNN
+F 1 "GND" H 2200 5750 50  0000 C CNN
+F 2 "" H 2200 5900 50  0000 C CNN
+F 3 "" H 2200 5900 50  0000 C CNN
+	1    2200 5900
+	1    0    0    -1
+$EndComp
+Wire Wire Line
+	2200 5850 2200 5900
+$Comp
+L C_Small C4
+U 1 1 57AC090F
+P 4850 7450
+F 0 "C4" H 4860 7520 50  0000 L CNN
+F 1 "0.1uF" H 4860 7370 50  0000 L CNN
+F 2 "Capacitors_ThroughHole:C_Disc_D3_P2.5" H 4850 7450 50  0001 C CNN
+F 3 "" H 4850 7450 50  0000 C CNN
+	1    4850 7450
+	1    0    0    -1
+$EndComp
+Wire Wire Line
+	5250 7400 5250 7600
+Connection ~ 5250 7600
+$Comp
+L +Vin #PWR035
+U 1 1 57AC0EE8
+P 4850 7350
+F 0 "#PWR035" H 4850 7200 50  0001 C CNN
+F 1 "+Vin" H 4850 7490 50  0000 C CNN
+F 2 "" H 4850 7350 50  0000 C CNN
+F 3 "" H 4850 7350 50  0000 C CNN
+	1    4850 7350
+	1    0    0    -1
+$EndComp
+Wire Wire Line
+	5250 7600 4850 7600
+Wire Wire Line
+	4850 7600 4850 7550
+$Comp
+L +3V3 #PWR036
+U 1 1 57AC16EA
+P 1950 3450
+F 0 "#PWR036" H 1950 3300 50  0001 C CNN
+F 1 "+3V3" H 1950 3590 50  0000 C CNN
+F 2 "" H 1950 3450 50  0000 C CNN
+F 3 "" H 1950 3450 50  0000 C CNN
+	1    1950 3450
+	1    0    0    -1
+$EndComp
+Connection ~ 1950 3600
+Wire Wire Line
+	1850 3750 1850 3600
+Wire Wire Line
+	1850 3600 2050 3600
+Wire Wire Line
+	2050 3600 2050 3750
+$Comp
+L C_Small C2
+U 1 1 57AC16F4
+P 2200 3550
+F 0 "C2" H 2210 3620 50  0000 L CNN
+F 1 "0.1uF" H 2210 3470 50  0000 L CNN
+F 2 "Capacitors_ThroughHole:C_Disc_D3_P2.5" H 2200 3550 50  0001 C CNN
+F 3 "" H 2200 3550 50  0000 C CNN
+	1    2200 3550
+	1    0    0    -1
+$EndComp
+Wire Wire Line
+	1950 3600 1950 3450
+Wire Wire Line
+	1950 3450 2200 3450
+Connection ~ 1950 3450
+Wire Wire Line
+	2200 3650 2200 3700
+$Comp
+L GND #PWR037
+U 1 1 57AC1742
+P 2200 3700
+F 0 "#PWR037" H 2200 3450 50  0001 C CNN
+F 1 "GND" H 2200 3550 50  0000 C CNN
+F 2 "" H 2200 3700 50  0000 C CNN
+F 3 "" H 2200 3700 50  0000 C CNN
+	1    2200 3700
+	1    0    0    -1
+$EndComp
+$Comp
+L CP C5
+U 1 1 57AC1C88
+P 6450 1400
+F 0 "C5" H 6475 1500 50  0000 L CNN
+F 1 "10uF" H 6475 1300 50  0000 L CNN
+F 2 "Capacitors_ThroughHole:C_Radial_D5_L6_P2.5" H 6488 1250 50  0001 C CNN
+F 3 "" H 6450 1400 50  0000 C CNN
+	1    6450 1400
+	1    0    0    -1
+$EndComp
+Connection ~ 6100 1600
+Wire Wire Line
+	6450 1600 6450 1550
+Wire Wire Line
+	6450 1150 6450 1250
+Connection ~ 6250 1150
 $EndSCHEMATC
